File: CANBusTriple_f.brd (EAGLE design)
At the start: 50.2 x 49.5 mm, 65 parts, among them IC4 MCP1703CB, IC6 IC_MEM_23LC1024, Q1 BSS138, Q2 BSS138, U1 BLE112

Commit message: Adding MCP2551 sleep lines - Rs
Connections:
- net N$12: now also CAN-CNT-3.10
- net N$3: now also CAN-CNT-1.10
- net N$4: now also CAN-CNT-2.10
Routing:
- net N$4: track 13.8 -> 31.2 mm, vias 0 -> 3
- net N$12: track 2.59 -> 16.8 mm, vias 0 -> 1
- net N$3: track 8.08 -> 19.4 mm, vias 0 -> 1
- net CAN2LOW: track 53.9 -> 55.3 mm
- net CAN2HIGH: track 55.6 -> 57.0 mm
- net MISO: track 71.1 -> 70.2 mm
Changed lines of the file:
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@@
 <wire x1="2.4384" y1="6.096" x2="5.3594" y2="6.096" width="0.2032" layer="16"/>
 <wire x1="5.3594" y1="6.096" x2="6.3246" y2="7.0612" width="0.2032" layer="16"/>
-<via x="11.811" y="9.144" extent="1-16" drill="0.3302"/>
+<via x="12.6238" y="9.9568" extent="1-16" drill="0.3302"/>
 <wire x1="6.3246" y1="7.0612" x2="6.3246" y2="7.8486" width="0.2032" layer="16"/>
 <wire x1="6.3246" y1="7.8486" x2="6.858" y2="8.382" width="0.2032" layer="16"/>
@@
 <wire x1="37.8468" y1="16.6624" x2="38.7096" y2="17.5252" width="0.1524" layer="1"/>
 <wire x1="15.5" y1="11.436" x2="14.8368" y2="10.7728" width="0.1524" layer="1"/>
-<wire x1="14.8368" y1="10.7728" x2="12.3984" y2="10.7728" width="0.1524" layer="1"/>
-<wire x1="12.3984" y1="10.7728" x2="11.7856" y2="10.16" width="0.1524" layer="1"/>
-<wire x1="11.7856" y1="10.16" x2="11.7856" y2="9.1694" width="0.1524" layer="1"/>
-<wire x1="11.7856" y1="9.1694" x2="11.811" y2="9.144" width="0.1524" layer="1"/>
 <wire x1="15.5" y1="12.25" x2="15.5" y2="11.7968" width="0.1524" layer="16"/>
 <wire x1="15.5" y1="11.436" x2="15.5" y2="11.7968" width="0.1524" layer="1"/>
 <wire x1="26.04" y1="13.75" x2="26.27" y2="13.98" width="0.1524" layer="16"/>
 <wire x1="26.5" y1="13.75" x2="26.27" y2="13.98" width="0.1524" layer="16"/>
-<wire x1="7.239" y1="9.525" x2="11.43" y2="9.525" width="0.2032" layer="16"/>
-<wire x1="11.43" y1="9.525" x2="11.811" y2="9.144" width="0.2032" layer="16"/>
+<wire x1="7.239" y1="9.525" x2="12.2428" y2="9.525" width="0.2032" layer="16"/>
+<wire x1="12.2428" y1="9.525" x2="12.6238" y2="9.9568" width="0.2032" layer="16"/>
+<wire x1="14.8368" y1="10.7728" x2="13.4398" y2="10.7728" width="0.1524" layer="1"/>
+<wire x1="13.4398" y1="10.7728" x2="12.6238" y2="9.9568" width="0.1524" layer="1"/>
 </signal>
 <signal name="N$3">
@@
 <wire x1="20.32" y1="6.096" x2="21.402" y2="6.096" width="0.254" layer="1"/>
 <wire x1="21.402" y1="6.096" x2="21.5392" y2="6.2332" width="0.254" layer="1"/>
+<contactref element="CAN-CNT-1" pad="10"/>
+<wire x1="7.3216" y1="14.7879" x2="7.3216" y2="13.4048" width="0.1524" layer="16"/>
+<wire x1="7.3216" y1="13.4048" x2="8.128" y2="12.5984" width="0.1524" layer="16"/>
+<via x="8.128" y="12.5984" extent="1-16" drill="0.3302"/>
+<wire x1="8.128" y1="12.5984" x2="10.16" y2="10.5664" width="0.1524" layer="1"/>
+<wire x1="10.16" y1="10.5664" x2="10.5664" y2="10.5664" width="0.1524" layer="1"/>
+<wire x1="10.5664" y1="10.5664" x2="12.192" y2="8.9408" width="0.1524" layer="1"/>
+<wire x1="12.192" y1="8.9408" x2="15.1152" y2="8.9408" width="0.1524" layer="1"/>
+<wire x1="15.1152" y1="8.9408" x2="15.3414" y2="9.167" width="0.1524" layer="1"/>
 </signal>
 <signal name="N$4">
@@
 <wire x1="35.3568" y1="4.6076" x2="34.4068" y2="4.6076" width="0.254" layer="1"/>
 <wire x1="34.4068" y1="4.6076" x2="33.7312" y2="5.2832" width="0.254" layer="1"/>
-<wire x1="33.7312" y1="5.2832" x2="33.7312" y2="10.5664" width="0.254" layer="1"/>
-<wire x1="33.7312" y1="10.5664" x2="33.3248" y2="10.9728" width="0.254" layer="1"/>
-<wire x1="33.3248" y1="10.9728" x2="29.2608" y2="10.9728" width="0.254" layer="1"/>
-<wire x1="29.2608" y1="10.9728" x2="28.8544" y2="10.5664" width="0.254" layer="1"/>
-<wire x1="28.8544" y1="10.5664" x2="28.8544" y2="9.2024" width="0.254" layer="1"/>
+<wire x1="33.7312" y1="5.2832" x2="33.7312" y2="10.16" width="0.254" layer="1"/>
+<wire x1="33.7312" y1="10.16" x2="33.3248" y2="10.5664" width="0.254" layer="1"/>
+<wire x1="33.3248" y1="10.5664" x2="29.2608" y2="10.5664" width="0.254" layer="1"/>
+<wire x1="29.2608" y1="10.5664" x2="28.8544" y2="10.16" width="0.254" layer="1"/>
+<wire x1="28.8544" y1="10.16" x2="28.8544" y2="9.2024" width="0.254" layer="1"/>
 <wire x1="28.8544" y1="9.2024" x2="28.819" y2="9.167" width="0.254" layer="1"/>
+<contactref element="CAN-CNT-2" pad="10"/>
+<wire x1="20.0184" y1="14.7879" x2="20.0184" y2="15.1416" width="0.1524" layer="16"/>
+<wire x1="20.0184" y1="15.1416" x2="21.1328" y2="16.256" width="0.1524" layer="16"/>
+<via x="21.1328" y="16.256" extent="1-16" drill="0.3302"/>
+<wire x1="21.1328" y1="16.256" x2="21.9456" y2="15.4432" width="0.1524" layer="1"/>
+<wire x1="21.9456" y1="15.4432" x2="21.9456" y2="8.9408" width="0.1524" layer="1"/>
+<wire x1="21.9456" y1="8.9408" x2="22.7584" y2="8.128" width="0.1524" layer="1"/>
+<wire x1="22.7584" y1="8.128" x2="25.1968" y2="8.128" width="0.1524" layer="1"/>
+<wire x1="25.1968" y1="8.128" x2="25.6032" y2="7.7216" width="0.1524" layer="1"/>
+<via x="25.6032" y="7.7216" extent="1-16" drill="0.3302"/>
+<wire x1="25.6032" y1="7.7216" x2="28.0416" y2="7.7216" width="0.1524" layer="16"/>
+<via x="28.0416" y="7.7216" extent="1-16" drill="0.3302"/>
+<wire x1="28.8544" y1="9.1316" x2="28.819" y2="9.167" width="0.1524" layer="1"/>
+<wire x1="28.8544" y1="9.1316" x2="28.8544" y2="8.128" width="0.1524" layer="1"/>
+<wire x1="28.8544" y1="8.128" x2="28.448" y2="7.7216" width="0.1524" layer="1"/>
+<wire x1="28.448" y1="7.7216" x2="28.0416" y2="7.7216" width="0.1524" layer="1"/>
 </signal>
 <signal name="N$18">
@@
 <via x="20.8264" y="17.0688" extent="1-16" drill="0.3302"/>
 <wire x1="31.359" y1="9.167" x2="31.359" y2="7.7878" width="0.1524" layer="1"/>
-<wire x1="31.359" y1="7.7878" x2="30.8864" y2="7.3152" width="0.1524" layer="1"/>
-<wire x1="30.8864" y1="7.3152" x2="28.0416" y2="7.3152" width="0.1524" layer="1"/>
-<wire x1="28.0416" y1="7.3152" x2="26.8224" y2="8.5344" width="0.1524" layer="1"/>
-<wire x1="26.8224" y1="8.5344" x2="26.8224" y2="9.2472" width="0.1524" layer="1"/>
+<wire x1="27.6352" y1="6.5024" x2="26.8224" y2="7.3152" width="0.1524" layer="1"/>
+<wire x1="26.8224" y1="7.3152" x2="26.8224" y2="9.2472" width="0.1524" layer="1"/>
 <wire x1="26.8224" y1="9.2472" x2="25.6032" y2="10.4664" width="0.1524" layer="1"/>
 <wire x1="25.6032" y1="10.4664" x2="25.6032" y2="17.4752" width="0.1524" layer="1"/>
@@
 <wire x1="20.32" y1="17.3252" x2="20.57" y2="17.3252" width="0.1524" layer="16"/>
 <wire x1="20.57" y1="17.3252" x2="20.8264" y2="17.0688" width="0.1524" layer="16"/>
+<wire x1="27.6352" y1="6.5024" x2="29.2608" y2="6.5024" width="0.1524" layer="1"/>
+<wire x1="29.2608" y1="6.5024" x2="30.48" y2="7.7216" width="0.1524" layer="1"/>
+<wire x1="30.48" y1="7.7216" x2="31.2928" y2="7.7216" width="0.1524" layer="1"/>
+<wire x1="31.2928" y1="7.7216" x2="31.359" y2="7.7878" width="0.1524" layer="1"/>
 </signal>
 <signal name="N$40">
@@
 <via x="20.7264" y="18.0316" extent="1-16" drill="0.3302"/>
 <wire x1="30.089" y1="9.167" x2="30.089" y2="8.1434" width="0.1524" layer="1"/>
-<wire x1="30.089" y1="8.1434" x2="29.6672" y2="7.7216" width="0.1524" layer="1"/>
-<wire x1="29.6672" y1="7.7216" x2="28.1416" y2="7.7216" width="0.1524" layer="1"/>
-<wire x1="28.1416" y1="7.7216" x2="27.2288" y2="8.6344" width="0.1524" layer="1"/>
-<wire x1="27.2288" y1="8.6344" x2="27.2288" y2="9.3472" width="0.1524" layer="1"/>
+<wire x1="28.8544" y1="6.9088" x2="27.7352" y2="6.9088" width="0.1524" layer="1"/>
+<wire x1="27.7352" y1="6.9088" x2="27.2288" y2="7.4152" width="0.1524" layer="1"/>
+<wire x1="27.2288" y1="7.4152" x2="27.2288" y2="9.3472" width="0.1524" layer="1"/>
 <wire x1="27.2288" y1="9.3472" x2="26.0096" y2="10.5664" width="0.1524" layer="1"/>
 <wire x1="26.0096" y1="10.5664" x2="26.0096" y2="17.8816" width="0.1524" layer="1"/>
@@
 <wire x1="25.1968" y1="18.6944" x2="21.3892" y2="18.6944" width="0.1524" layer="1"/>
 <wire x1="21.3892" y1="18.6944" x2="20.7264" y2="18.0316" width="0.1524" layer="1"/>
+<wire x1="28.8544" y1="6.9088" x2="30.089" y2="8.1434" width="0.1524" layer="1"/>
 </signal>
 <signal name="N$11">
@@
 <wire x1="37.9078" y1="9.167" x2="35.4458" y2="9.167" width="0.254" layer="1"/>
 <wire x1="35.4458" y1="9.167" x2="35.3568" y2="9.078" width="0.254" layer="1"/>
+<contactref element="CAN-CNT-3" pad="10"/>
+<wire x1="32.42" y1="14.7879" x2="32.42" y2="15.9416" width="0.1524" layer="16"/>
+<wire x1="32.42" y1="15.9416" x2="32.1056" y2="16.256" width="0.1524" layer="16"/>
+<via x="32.1056" y="16.256" extent="1-16" drill="0.3302"/>
+<wire x1="32.1056" y1="16.256" x2="30.8864" y2="16.256" width="0.1524" layer="1"/>
+<wire x1="30.8864" y1="16.256" x2="30.48" y2="15.8496" width="0.1524" layer="1"/>
+<wire x1="30.48" y1="15.8496" x2="30.48" y2="11.6292" width="0.1524" layer="1"/>
+<wire x1="30.48" y1="11.6292" x2="30.8864" y2="11.2228" width="0.1524" layer="1"/>
+<wire x1="30.8864" y1="11.2228" x2="34.294" y2="11.2228" width="0.1524" layer="1"/>
+<wire x1="34.294" y1="11.2228" x2="35.3568" y2="10.16" width="0.1524" layer="1"/>
+<wire x1="35.3568" y1="10.16" x2="35.3568" y2="9.078" width="0.1524" layer="1"/>
 </signal>
 <signal name="N$13">

Commit message: switching to single direction LLC to remove MOSFETs
Parts:
- removed A8: (no value), wirepad:SMD1,27-2,54
- removed Q2: BSS138, SparkFun-DiscreteSemi:SOT23
- added R13: 10k, resistor:M0805
- R9: value 10k -> 5k
Connections:
- net CAN1_INT: no longer Q2.3
- net GND: now also R13.1; no longer Q2.2, R9.1
- net N$29: now also R13.2, R9.1; no longer Q2.1, R9.2
- net N$36: now also R9.2; no longer A8.1
Routing:
- net N$29: track 21.2 -> 0.00 mm, vias 2 -> 0
- net CAN1_INT: track 38.6 -> 34.2 mm
Changed lines of the file:
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@@
 <element name="U1" library="ble112" package="SF-BLUEGIGA_BLE112-A" value="BLE112" x="9.57" y="27.54" smashed="yes" rot="R90">
 <attribute name="NAME" x="8.278" y="30.592" size="1.016" layer="25" rot="SR0"/>
-<attribute name="VALUE" x="8.278" y="28.592" size="1.016" layer="27" rot="SR0"/>
+<attribute name="VALUE" x="7.8716" y="25.7472" size="1.016" layer="27" rot="SR0"/>
 </element>
 <element name="F1" library="rcl" package="L1812" value="POLYFUSE" x="11.642" y="46.0958" smashed="yes" rot="MR180">
@@
 <attribute name="VALUE" x="4.5448" y="39.4888" size="0.8128" layer="28" font="vector" rot="MR270"/>
 </element>
-<element name="A8" library="wirepad" package="SMD1,27-2,54" value="" x="27.754234375" y="31.98656875" smashed="yes" rot="MR45">
-<attribute name="VALUE" x="27.754234375" y="31.98656875" size="0.0254" layer="28" rot="MR45"/>
-<attribute name="NAME" x="26.216465625" y="32.568628125" size="0.8128" layer="26" rot="MR135"/>
-</element>
-<element name="Q2" library="SparkFun-DiscreteSemi" package="SOT23" value="BSS138" x="11.3792" y="15.0368" rot="R270">
-<attribute name="PROD_ID" value="TRANS-08345" x="11.3792" y="15.0368" size="0.8128" layer="27" rot="R270" display="off"/>
-</element>
-<element name="R9" library="resistor" package="M0805" value="10k" x="7.7216" y="15.0368" rot="R90"/>
+<element name="R9" library="resistor" package="M0805" value="5k" x="7.7216" y="15.0368" rot="R90"/>
+<element name="R13" library="resistor" package="M0805" value="10k" x="10.16" y="15.0368" rot="R90"/>
 </elements>
 <signals>
@@
 <wire x1="21.7456" y1="24.184" x2="22.352" y2="24.7904" width="0.1524" layer="1"/>
 <wire x1="22.352" y1="24.7904" x2="22.352" y2="25.6032" width="0.1524" layer="1"/>
-<contactref element="Q2" pad="3"/>
-<wire x1="12.4792" y1="15.0368" x2="13.4112" y2="15.0368" width="0.2" layer="1"/>
-<wire x1="13.4112" y1="15.0368" x2="15.8496" y2="17.4752" width="0.2" layer="1"/>
 </signal>
 <signal name="N$24">
@@
 <contactref element="U$1" pad="28"/>
 <wire x1="26.880578125" y1="31.0724125" x2="26.880578125" y2="30.879021875" width="0.1524" layer="1"/>
-<contactref element="A8" pad="1"/>
 <wire x1="26.880578125" y1="31.0724125" x2="26.880578125" y2="31.234621875" width="0.1524" layer="1"/>
 <wire x1="26.880578125" y1="31.234621875" x2="26.0096" y2="32.1056" width="0.1524" layer="1"/>
 <via x="26.0096" y="32.1056" extent="1-16" drill="0.3302" diameter="0.3302"/>
 <wire x1="26.0096" y1="32.1056" x2="27.635203125" y2="32.1056" width="0.1524" layer="16"/>
-<wire x1="27.635203125" y1="32.1056" x2="27.754234375" y2="31.98656875" width="0.1524" layer="16"/>
+<contactref element="R9" pad="2"/>
+<wire x1="7.7216" y1="15.9868" x2="26.880578125" y2="30.879021875" width="0" layer="19" extent="1-1"/>
 </signal>
 <signal name="N$37">
@@
 <via x="4.4208" y="26.1848" extent="1-16" drill="0.3302"/>
 <via x="9.2976" y="27.8104" extent="1-16" drill="0.3302"/>
-<via x="10.3004" y="12.9252" extent="1-16" drill="0.3302"/>
+<via x="9.894" y="12.5188" extent="1-16" drill="0.3302"/>
 <via x="25.96" y="33.9064" extent="1-16" drill="0.3302"/>
 <wire x1="3.2732" y1="20.2974" x2="2.4384" y2="20.1974" width="0.4064" layer="16"/>
@@
 <via x="39.928" y="33.1272" extent="1-16" drill="0.3302"/>
 <contactref element="D2" pad="A"/>
-<contactref element="R9" pad="1"/>
-<contactref element="Q2" pad="2"/>
+<contactref element="R13" pad="1"/>
+<wire x1="12.67" y1="21.49" x2="17.4256" y2="20.9016" width="0" layer="19" extent="1-1"/>
 </signal>
 <signal name="VBUS">
@@
 </signal>
 <signal name="N$29">
-<contactref element="R9" pad="2"/>
-<contactref element="Q2" pad="1"/>
 <contactref element="U1" pad="P1_0"/>
-<wire x1="7.7216" y1="15.9868" x2="10.2792" y2="15.9868" width="0.5" layer="1"/>
-<wire x1="10.2792" y1="15.9868" x2="11.11" y2="15.9868" width="0.2" layer="1"/>
-<wire x1="11.11" y1="15.9868" x2="11.3792" y2="16.256" width="0.2" layer="1"/>
-<wire x1="11.3792" y1="16.256" x2="12.5984" y2="16.256" width="0.2" layer="1"/>
-<wire x1="12.5984" y1="16.256" x2="13.4112" y2="17.0688" width="0.2" layer="1"/>
-<via x="13.4112" y="17.0688" extent="1-16" drill="0.3302" diameter="0.3302"/>
-<wire x1="13.4112" y1="17.0688" x2="13.4112" y2="17.5112" width="0.2" layer="16"/>
-<wire x1="13.4112" y1="17.5112" x2="14.8" y2="18.9" width="0.2" layer="16"/>
-<wire x1="14.8" y1="18.9" x2="14.8" y2="21.7936" width="0.2" layer="16"/>
-<wire x1="14.8" y1="21.7936" x2="16.85" y2="23.8436" width="0.2" layer="16"/>
-<wire x1="16.85" y1="23.8436" x2="16.85" y2="27.4476" width="0.2" layer="16"/>
-<wire x1="16.85" y1="27.4476" x2="16.256" y2="28.0416" width="0.2" layer="16"/>
-<via x="16.256" y="28.0416" extent="1-16" drill="0.3302" diameter="0.3302"/>
-<wire x1="16.256" y1="28.0416" x2="18.5216" y2="28.0416" width="0.2" layer="1"/>
-<wire x1="18.5216" y1="28.0416" x2="18.62" y2="28.14" width="0.2" layer="1"/>
+<contactref element="R13" pad="2"/>
+<contactref element="R9" pad="1"/>
+<wire x1="10.16" y1="15.9868" x2="18.62" y2="28.14" width="0" layer="19" extent="1-1"/>
+<wire x1="7.7216" y1="14.0868" x2="10.16" y2="15.9868" width="0" layer="19" extent="1-1"/>
 </signal>
 </signals>

Commit message: switched UART Tx from MCU to BLE to simple unidirectional logic level conversion
Parts:
- removed Q1: BSS138, SparkFun-DiscreteSemi:SOT23
- R11: value 10k -> 5k
Connections:
- net +3V: no longer Q1.1, R10.2
- net +5V: no longer R11.2
- net GND: now also R10.1
- net N$19: now also R11.2; no longer Q1.3, R11.1
- net N$38: now also R10.2, R11.1; no longer Q1.2, R10.1
Routing:
- net +3V: track 64.9 -> 58.8 mm
- net N$19: track 7.87 -> 4.28 mm
- net N$38: track 38.3 -> 36.0 mm
- net +5V: track 260.9 -> 259.0 mm
Changed lines of the file:
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@@
 <attribute name="NAME" x="10.737" y="46.6908" size="1.27" layer="26" rot="MR180"/>
-</element>
-<element name="Q1" library="SparkFun-DiscreteSemi" package="SOT23" value="BSS138" x="30.9896" y="36.1508" smashed="yes" rot="MR90">
-<attribute name="PROD_ID" value="TRANS-08345" x="30.9896" y="36.1508" size="1.778" layer="28" rot="MR90" display="off"/>
-<attribute name="NAME" x="31.9548" y="34.8808" size="0.4064" layer="26" rot="MR90"/>
-<attribute name="VALUE" x="30.7991" y="35.1348" size="0.4064" layer="28" rot="MR90"/>
 </element>
 <element name="R10" library="resistor" package="M0805" value="10k" x="27.9872" y="35.838" smashed="yes" rot="MR270">
 <attribute name="NAME" x="26.9712" y="36.854" size="1.016" layer="26" rot="MR270"/>
 </element>
-<element name="R11" library="resistor" package="M0805" value="10k" x="29.75" y="39.1268" smashed="yes" rot="MR0">
+<element name="R11" library="resistor" package="M0805" value="5k" x="29.75" y="39.1268" smashed="yes" rot="MR0">
 <attribute name="NAME" x="30.766" y="40.1428" size="1.016" layer="26" rot="MR0"/>
 </element>
@@
 <contactref element="D2" pad="A"/>
 <contactref element="R13" pad="1"/>
-<wire x1="12.67" y1="21.49" x2="17.4256" y2="20.9016" width="0" layer="19" extent="1-1"/>
+<contactref element="R10" pad="1"/>
+<wire x1="29.70900625" y1="33.9008375" x2="27.9872" y2="36.788" width="0" layer="19" extent="1-16"/>
+<wire x1="17.4256" y1="20.9016" x2="12.67" y2="21.49" width="0" layer="19" extent="1-1"/>
 </signal>
 <signal name="VBUS">
@@
 <contactref element="U$1" pad="24"/>
 <contactref element="U$1" pad="44"/>
-<contactref element="R11" pad="2"/>
 <wire x1="48.746" y1="22.098" x2="48.746" y2="21.9676" width="0.5" layer="1"/>
 <wire x1="48.746" y1="21.9676" x2="49.1744" y2="21.5392" width="0.5" layer="1"/>
@@
 <wire x1="15.0368" y1="36.6388" x2="15" y2="36.6388" width="0.4064" layer="1"/>
 <wire x1="15" y1="36.6388" x2="15" y2="36.7284" width="0.4064" layer="1"/>
-<wire x1="28.8" y1="39.1268" x2="28.8" y2="40.992" width="0.5" layer="16"/>
 <wire x1="28.8" y1="40.992" x2="28.448" y2="41.0464" width="0.5" layer="16"/>
 <via x="28.448" y="41.0464" extent="1-16" drill="0.5"/>
@@
 <contactref element="U1" pad="AVDD2"/>
 <contactref element="U1" pad="DVDD"/>
-<contactref element="R10" pad="2"/>
-<contactref element="Q1" pad="1"/>
 <contactref element="IC4" pad="2"/>
 <contactref element="C4" pad="1"/>
@@
 <wire x1="4.7298" y1="22.352" x2="4.7988" y2="22.283" width="0.3" layer="16"/>
 <wire x1="4.038" y1="18.3" x2="4" y2="18.262" width="0.5" layer="1"/>
-<wire x1="29.8896" y1="35.2008" x2="28.3" y2="35.2008" width="0.5" layer="16"/>
-<wire x1="28.3" y1="35.2008" x2="27.9872" y2="34.888" width="0.5" layer="16"/>
-<wire x1="27.9872" y1="34.888" x2="23.9152" y2="34.888" width="0.33" layer="16"/>
 <wire x1="23.9152" y1="34.888" x2="21.9456" y2="32.9184" width="0.33" layer="16"/>
 <via x="21.9456" y="32.9184" extent="1-16" drill="0.3302"/>
@@
 <signal name="N$19">
 <contactref element="U$1" pad="21"/>
-<contactref element="Q1" pad="3"/>
-<contactref element="R11" pad="1"/>
 <wire x1="32.820275" y1="33.335153125" x2="32.928753125" y2="33.335153125" width="0.2032" layer="1"/>
 <wire x1="32.928753125" y1="33.335153125" x2="33.5312" y2="33.9312" width="0.2032" layer="1"/>
@@
 <via x="32.1056" y="35.0568" extent="1-16" drill="0.3302"/>
 <wire x1="32.1056" y1="35.0568" x2="32.1056" y2="36.1348" width="0.2032" layer="16"/>
-<wire x1="32.1056" y1="36.1348" x2="32.0896" y2="36.1508" width="0.2032" layer="16"/>
-<wire x1="30.7" y1="39.1268" x2="30.7" y2="38.7944" width="0.5" layer="16"/>
-<wire x1="30.7" y1="38.7944" x2="32.1056" y2="37.3888" width="0.5" layer="16"/>
-<wire x1="32.1056" y1="37.3888" x2="32.1056" y2="36.1668" width="0.5" layer="16"/>
-<wire x1="32.1056" y1="36.1668" x2="32.0896" y2="36.1508" width="0.5" layer="16"/>
+<contactref element="R11" pad="2"/>
+<wire x1="32.1056" y1="36.1348" x2="28.8" y2="39.1268" width="0" layer="19" extent="16-16"/>
 </signal>
 <signal name="N$44">
@@
 <signal name="N$38">
 <contactref element="U1" pad="P1_7"/>
-<contactref element="R10" pad="1"/>
-<contactref element="Q1" pad="2"/>
-<wire x1="29.8896" y1="37.1008" x2="28.3" y2="37.1008" width="0.5" layer="16"/>
-<wire x1="28.3" y1="37.1008" x2="27.9872" y2="36.788" width="0.5" layer="16"/>
 <wire x1="20.5264" y1="21.5392" x2="18.088" y2="19.1008" width="0.1524" layer="1"/>
 <wire x1="18.088" y1="19.1008" x2="14.224" y2="19.1008" width="0.1524" layer="1"/>
@@
 <wire x1="22.3084" y1="34.544" x2="24.7468" y2="36.9824" width="0.1524" layer="16"/>
 <wire x1="24.7468" y1="36.9824" x2="27.7928" y2="36.9824" width="0.1524" layer="16"/>
-<wire x1="27.7928" y1="36.9824" x2="27.9872" y2="36.788" width="0.1524" layer="16"/>
 <wire x1="13.4112" y1="18.288" x2="10.16" y2="18.288" width="0.1524" layer="1"/>
 <wire x1="10.16" y1="18.288" x2="8.9408" y2="19.5072" width="0.1524" layer="1"/>
 <wire x1="8.9408" y1="19.5072" x2="8.9408" y2="21.4692" width="0.1524" layer="1"/>
 <wire x1="8.9408" y1="21.4692" x2="8.92" y2="21.49" width="0.1524" layer="1"/>
+<contactref element="R10" pad="2"/>
+<contactref element="R11" pad="1"/>
+<wire x1="27.7928" y1="36.9824" x2="30.7" y2="39.1268" width="0" layer="19" extent="16-16"/>
+<wire x1="27.9872" y1="34.888" x2="27.7928" y2="36.9824" width="0" layer="19" extent="16-16"/>
 </signal>
 <signal name="N$45">

Commit message: Last sleep mode tweak, added line from BT LE to CAN1INT to wake the MCU up via BT
Parts:
- added Q1: MOSFET-NCHANNEL2N7002PW, SparkFun-DiscreteSemi:SOT323
- L1: value 47uH -> 68uH
- moved R13 22.2 mm to (22.8, 33.3), turned to 180 degrees
- moved R9 22.1 mm to (22.8, 31.3), turned to 0 degrees
- moved D3 2.02 mm to (12.5, 43.7), flipped to the bottom, turned to 180 degrees
- moved R10 1.83 mm to (29.7, 36.6), turned to 0 degrees
- moved F1 0.57 mm to (11.2, 46.5)
- moved CAN1-TRM 0.41 mm to (16.9, 45.0)
- moved R11 0.14 mm to (29.7, 39.0), turned to 180 degrees
Connections:
- new net N$33: Q1.1, U1.P0_1
- net +5V: no longer L1.2
- net CAN1_INT: now also Q1.3
- net GND: now also Q1.2
Routing:
- net N$33: track 0.00 -> 25.3 mm, vias 0 -> 2
- net +5V: track 259.0 -> 248.7 mm, vias 12 -> 11
- net +3V: track 58.8 -> 50.8 mm, vias 6 -> 5
- net N$29: track 0.00 -> 7.65 mm
- net N$22: track 7.25 -> 2.90 mm, vias 1 -> 0
- net N$19: track 4.28 -> 8.17 mm
- net CAN1_INT: track 34.2 -> 37.6 mm
- net N$38: track 36.0 -> 39.3 mm
- net GND: track 34.9 -> 36.9 mm
- net SUPPLY: track 19.1 -> 18.1 mm
- net N$36: track 3.21 -> 3.89 mm, vias 1 -> 0

Commit message: Fix missing trace on inductor
Connections:
- net +5V: now also L1.2
Routing:
- net +5V: track 248.7 -> 251.5 mm
Changed lines of the file:
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@@
 <wire x1="11.3792" y1="36.9824" x2="10.5664" y2="37.7952" width="0.5" layer="1"/>
 <wire x1="10.5664" y1="37.7952" x2="9.7536" y2="37.7952" width="0.5" layer="1"/>
+<contactref element="L1" pad="2"/>
+<wire x1="7.6396" y1="39.0144" x2="7.6396" y2="38.69" width="0.5" layer="1"/>
+<wire x1="7.6396" y1="38.69" x2="8.5344" y2="37.7952" width="0.5" layer="1"/>
+<wire x1="8.5344" y1="37.7952" x2="9.7536" y2="37.7952" width="0.5" layer="1"/>
 </signal>
 <signal name="CAN1HIGH">
