File: CANBusTriple_f.brd (EAGLE design)
At the start: 50.2 x 49.5 mm, 64 parts, among them IC4 MCP1703CB, IC6 IC_MEM_23LC1024, Q1 MOSFET-NCHANNEL2N7002PW, U1 BLE112

Commit message: switched to LM3480IM3-5.0
Parts:
- removed C11: .01 uF, resistor:C0603
- removed D3: (no value), adafruit:SOD-323F
- removed IC5: (no value), lm2674:SO8
- removed L1: 68uH, inductor-bourns:SDR0604
- added IC1: LM3480, CustomParts_CBT:SOT23
- C1: value 22uF -> 0.1uF; device resistor:C0805 -> resistor:C0603
- C2: value 47uF -> 0.1uF; device resistor:C1206 -> resistor:C0603
- moved C3 14.7 mm to (12.2, 34.1), turned to 270 degrees
- moved C4 12.0 mm to (8.94, 31.3), turned to 180 degrees
- moved IC4 11.6 mm to (8.94, 34.5)
- moved D2 7.76 mm to (8.53, 42.7), turned to 0 degrees
- moved C2 2.93 mm to (7.72, 39.0), flipped to the top
- moved R10 2.03 mm to (29.7, 38.6)
- moved C1 1.74 mm to (7.72, 41.5), flipped to the top, turned to 0 degrees
- moved R11 1.63 mm to (29.7, 40.6)
- moved U1 1.22 mm to (9.57, 28.8)
- moved F1 1.15 mm to (12.0, 45.7)
- moved U$8 0.91 mm to (7.54, 47.3)
- moved R9 0.81 mm to (22.8, 32.1)
- moved R13 0.81 mm to (22.8, 34.1)
- moved CN1 0.46 mm to (35.7, 46.0)
- moved U$10 0.41 mm to (4.00, 18.7)
- renumbered U$11 to Q2, U$2 to Q0
Connections:
- removed net N$22: D3.C, F1.2
- removed net N$34: C11.1, IC5.1
- net +12V: now also F1.2; no longer D3.A
- net +5V: now also IC1.1; no longer IC5.4, L1.2
- net GND: now also IC1.3; no longer D2.A, IC5.6
- net N$15: now also D2.A, F1.1; no longer C11.2, D2.C, IC5.8, L1.1
- net SUPPLY: now also D2.C, IC1.2; no longer F1.1, IC5.7
Routing:
- net SUPPLY: track 18.1 -> 7.04 mm, vias 0 -> 1
- net +5V: track 251.5 -> 240.9 mm, vias 11 -> 10
- net N$15: track 13.0 -> 3.41 mm, vias 1 -> 0
- net N$34: track 8.56 -> 0.00 mm, vias 2 -> 0
- net +3V: track 50.8 -> 57.4 mm
- net GND: track 36.9 -> 31.7 mm, vias 23 -> 24
- net N$22: track 2.90 -> 0.00 mm
- net N$38: track 39.3 -> 41.9 mm
- net N$33: track 25.3 -> 27.4 mm
- net N$19: track 8.17 -> 10.2 mm
- net +12V: track 3.49 -> 4.82 mm
- net MCU_RESET: track 87.1 -> 85.9 mm
- net CAN1_INT: track 37.6 -> 36.4 mm
- net BLE-112-P1_3: track 1.02 -> 0.00 mm
- net BLE-112-P0_2: track 28.0 -> 29.0 mm
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
Commit message: switched to TPS70950 LDO Linear Regulator
Parts:
- removed D2: (no value), adafruit:SOD-323F
- removed F1: POLYFUSE, rcl:L1812
- C1: value 0.1uF -> 1uF
- C2: value 0.1uF -> 2.2uF
- IC1: value LM3480 -> TPS709-50; device CustomParts_CBT:SOT23 -> CustomParts_CBT:SOT23-5
- moved IC1 0.57 mm to (3.66, 39.8), turned to 180 degrees
- moved U$10 0.41 mm to (4.00, 19.1)
Connections:
- removed net N$15: D2.A, F1.1
- removed net SUPPLY: C1.1, D2.C, IC1.2
- net +12V: now also C1.1, IC1.1; no longer F1.2
- net +5V: now also IC1.5; no longer IC1.1
- net GND: now also IC1.2; no longer IC1.3
Routing:
- net SUPPLY: track 7.04 -> 0.00 mm, vias 1 -> 0
- net +12V: track 4.82 -> 10.8 mm, vias 0 -> 1
- net N$15: track 3.41 -> 0.00 mm
- net +5V: track 240.9 -> 241.8 mm
- net BLE-112-P0_2: track 29.0 -> 28.3 mm

Commit message: Some part name changes
Parts:
- renumbered CAN-CNT-1 to CC1, CAN-CNT-2 to CC2, CAN-CNT-3 to CC3, CAN-TRNS-1 to CT1, CAN-TRNS-2 to CT2, CAN-TRNS-3 to CT3, CAN1-TRM to R14, CAN2-TRM to R15, CAN3-TRM to R16
