File: CANBusTriple_f.sch (EAGLE design)
At the start: 61 parts, among them IC4 MCP1703CB, IC6 IC_MEM_23LC1024, Q1 BSS138, Q2 BSS138, U1 BLE112

Commit message: Adding MCP2551 sleep lines - Rs
Connections:
- net N$12: now also CAN-CNT-3D.RX1BF
- net N$3: now also CAN-CNT-1D.RX1BF
- net N$4: now also CAN-CNT-2D.RX1BF
Changed lines of the file:
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@@
 <pinref part="R1" gate="G$1" pin="2"/>
 <wire x1="289.56" y1="86.36" x2="292.1" y2="86.36" width="0.1524" layer="91"/>
+<pinref part="CAN-CNT-1" gate="D" pin="RX1BF"/>
+<wire x1="271.78" y1="76.2" x2="281.94" y2="76.2" width="0.1524" layer="91"/>
+<wire x1="281.94" y1="76.2" x2="281.94" y2="86.36" width="0.1524" layer="91"/>
+<wire x1="281.94" y1="86.36" x2="289.56" y2="86.36" width="0.1524" layer="91"/>
 </segment>
 </net>
@@
 <pinref part="R2" gate="G$1" pin="2"/>
 <wire x1="289.56" y1="48.26" x2="292.1" y2="48.26" width="0.1524" layer="91"/>
+<pinref part="CAN-CNT-2" gate="D" pin="RX1BF"/>
+<wire x1="271.78" y1="38.1" x2="281.94" y2="38.1" width="0.1524" layer="91"/>
+<wire x1="281.94" y1="38.1" x2="281.94" y2="48.26" width="0.1524" layer="91"/>
+<wire x1="281.94" y1="48.26" x2="289.56" y2="48.26" width="0.1524" layer="91"/>
 </segment>
 </net>
@@
 <pinref part="R5" gate="G$1" pin="2"/>
 <wire x1="294.64" y1="5.08" x2="297.18" y2="5.08" width="0.1524" layer="91"/>
-</segment>
-</net>
+<pinref part="CAN-CNT-3" gate="D" pin="RX1BF"/>
+<wire x1="281.94" y1="-5.08" x2="287.02" y2="-5.08" width="0.1524" layer="91"/>
+<wire x1="287.02" y1="-5.08" x2="287.02" y2="5.08" width="0.1524" layer="91"/>
+<wire x1="287.02" y1="5.08" x2="294.64" y2="5.08" width="0.1524" layer="91"/>
+</segment>
+</net>

Commit message: switching to single direction LLC to remove MOSFETs
Parts:
- removed A8: WIREPADSMD1,27-254, wirepad:WIREPADSMD1,27-254
- removed Q2: BSS138, SparkFun-DiscreteSemi:MOSFET-NCHANNELBSS123LT1G
- added R13: 10k, resistor:R-US_M0805
- R9: value 10k -> 5k
Connections:
- net CAN1_INT: no longer Q2.D
- net GND: now also R13.1; no longer Q2.S, R9.1
- net N$29: now also R13.2, R9.1; no longer Q2.G, R9.2
- net N$36: now also R9.2; no longer A8.P
Other:
- moved on the sheet: R9
Changed lines of the file:
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@@
 <part name="D3" library="adafruit" deviceset="DIODE" device="SOD-323F"/>
 <part name="D2" library="adafruit" deviceset="DIODE" device="SOD-323F"/>
-<part name="A8" library="wirepad" deviceset="WIREPAD" device="SMD1,27-254" value=""/>
-<part name="Q2" library="SparkFun-DiscreteSemi" deviceset="MOSFET-NCHANNEL" device="BSS123LT1G" value="BSS138"/>
 <part name="SUPPLY11" library="supply2" deviceset="GND" device=""/>
-<part name="R9" library="resistor" deviceset="R-US_" device="M0805" value="10k"/>
+<part name="R9" library="resistor" deviceset="R-US_" device="M0805" value="5k"/>
+<part name="R13" library="resistor" deviceset="R-US_" device="M0805" value="10k"/>
 </parts>
 <sheets>
@@
 <instance part="D3" gate="G$1" x="-20.32" y="93.98" rot="R270"/>
 <instance part="D2" gate="G$1" x="15.24" y="73.66" rot="R90"/>
-<instance part="A8" gate="G$1" x="165.1" y="144.78" rot="R270"/>
-<instance part="Q2" gate="G$1" x="208.28" y="-53.34" rot="R270"/>
-<instance part="SUPPLY11" gate="GND" x="200.66" y="-58.42"/>
-<instance part="R9" gate="G$1" x="200.66" y="-45.72" rot="R90"/>
+<instance part="SUPPLY11" gate="GND" x="175.26" y="-71.12"/>
+<instance part="R9" gate="G$1" x="175.26" y="-48.26" rot="R90"/>
+<instance part="R13" gate="G$1" x="175.26" y="-60.96" rot="R90"/>
 </instances>
 <busses>
@@
 <pinref part="CAN-CNT-1" gate="D" pin="INT"/>
 <wire x1="213.36" y1="96.52" x2="238.76" y2="96.52" width="0.1524" layer="91"/>
-<wire x1="213.36" y1="5.08" x2="213.36" y2="-53.34" width="0.1524" layer="91"/>
-<pinref part="Q2" gate="G$1" pin="D"/>
 </segment>
 </net>
@@
 <pinref part="U$1" gate="G$1" pin="PB4(ADC11)"/>
 <wire x1="134.62" y1="38.1" x2="165.1" y2="38.1" width="0.1524" layer="91"/>
-<wire x1="165.1" y1="38.1" x2="165.1" y2="142.24" width="0.1524" layer="91"/>
-<pinref part="A8" gate="G$1" pin="P"/>
+<wire x1="165.1" y1="38.1" x2="165.1" y2="-40.64" width="0.1524" layer="91"/>
+<pinref part="R9" gate="G$1" pin="2"/>
+<wire x1="165.1" y1="-40.64" x2="175.26" y2="-40.64" width="0.1524" layer="91"/>
+<wire x1="175.26" y1="-40.64" x2="175.26" y2="-43.18" width="0.1524" layer="91"/>
 </segment>
 </net>
@@
 </segment>
 <segment>
-<pinref part="R9" gate="G$1" pin="1"/>
+<pinref part="R13" gate="G$1" pin="1"/>
 <pinref part="SUPPLY11" gate="GND" pin="GND"/>
-<wire x1="200.66" y1="-50.8" x2="200.66" y2="-53.34" width="0.1524" layer="91"/>
-<pinref part="Q2" gate="G$1" pin="S"/>
-<wire x1="200.66" y1="-53.34" x2="200.66" y2="-55.88" width="0.1524" layer="91"/>
-<wire x1="203.2" y1="-53.34" x2="200.66" y2="-53.34" width="0.1524" layer="91"/>
+<wire x1="175.26" y1="-66.04" x2="175.26" y2="-68.58" width="0.1524" layer="91"/>
 </segment>
 </net>
@@
 <net name="N$29" class="0">
 <segment>
-<pinref part="R9" gate="G$1" pin="2"/>
-<pinref part="Q2" gate="G$1" pin="G"/>
-<wire x1="200.66" y1="-40.64" x2="208.28" y2="-40.64" width="0.1524" layer="91"/>
-<wire x1="208.28" y1="-40.64" x2="208.28" y2="-45.72" width="0.1524" layer="91"/>
-<wire x1="200.66" y1="-40.64" x2="190.5" y2="-40.64" width="0.1524" layer="91"/>
-<wire x1="190.5" y1="-40.64" x2="190.5" y2="-81.28" width="0.1524" layer="91"/>
-<wire x1="190.5" y1="-81.28" x2="114.3" y2="-81.28" width="0.1524" layer="91"/>
+<wire x1="167.64" y1="-81.28" x2="114.3" y2="-81.28" width="0.1524" layer="91"/>
 <pinref part="U1" gate="G$1" pin="P1_0"/>
 <wire x1="114.3" y1="-81.28" x2="114.3" y2="-63.5" width="0.1524" layer="91"/>
-</segment>
-</net>
+<wire x1="167.64" y1="-81.28" x2="167.64" y2="-55.88" width="0.1524" layer="91"/>
+<pinref part="R13" gate="G$1" pin="2"/>
+<wire x1="167.64" y1="-55.88" x2="175.26" y2="-55.88" width="0.1524" layer="91"/>
+<pinref part="R9" gate="G$1" pin="1"/>
+<wire x1="175.26" y1="-53.34" x2="175.26" y2="-55.88" width="0.1524" layer="91"/>
+<junction x="175.26" y="-55.88"/>
+</segment>
+</net>

Commit message: switched UART Tx from MCU to BLE to simple unidirectional logic level conversion
Parts:
- removed Q1: BSS138, SparkFun-DiscreteSemi:MOSFET-NCHANNELBSS123LT1G
- R11: value 10k -> 5k
Connections:
- net +3V: no longer Q1.G, R10.2
- net +5V: no longer R11.2
- net GND: now also R10.1
- net N$19: now also R11.2; no longer Q1.D, R11.1
- net N$38: now also R10.2, R11.1; no longer Q1.S, R10.1
Other:
- moved on the sheet: R10, R11
Changed lines of the file:
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@@
 <part name="F1" library="rcl" deviceset="L-EU" device="L1812" value="POLYFUSE"/>
 <part name="SUPPLY5" library="supply2" deviceset="GND" device=""/>
-<part name="Q1" library="SparkFun-DiscreteSemi" deviceset="MOSFET-NCHANNEL" device="BSS123LT1G" value="BSS138"/>
 <part name="R10" library="resistor" deviceset="R-US_" device="M0805" value="10k"/>
-<part name="R11" library="resistor" deviceset="R-US_" device="M0805" value="10k"/>
+<part name="R11" library="resistor" deviceset="R-US_" device="M0805" value="5k"/>
 <part name="BT" library="led" deviceset="LED" device="SMT1206"/>
 <part name="R12" library="resistor" deviceset="R-US_" device="M0805" value="10k"/>
@@
 <part name="R9" library="resistor" deviceset="R-US_" device="M0805" value="5k"/>
 <part name="R13" library="resistor" deviceset="R-US_" device="M0805" value="10k"/>
+<part name="SUPPLY14" library="supply2" deviceset="GND" device=""/>
 </parts>
 <sheets>
@@
 <instance part="F1" gate="G$1" x="-20.32" y="83.82" rot="R180"/>
 <instance part="SUPPLY5" gate="GND" x="66.04" y="-43.18"/>
-<instance part="Q1" gate="G$1" x="185.42" y="-22.86" rot="R270"/>
-<instance part="R10" gate="G$1" x="172.72" y="-17.78" rot="R90"/>
-<instance part="R11" gate="G$1" x="198.12" y="-17.78" rot="R90"/>
+<instance part="R10" gate="G$1" x="157.48" y="-20.32" rot="R90"/>
+<instance part="R11" gate="G$1" x="157.48" y="-7.62" rot="R90"/>
 <instance part="BT" gate="G$1" x="142.24" y="-58.42" rot="R90"/>
 <instance part="R12" gate="G$1" x="152.4" y="-63.5" rot="R90"/>
@@
 <instance part="R9" gate="G$1" x="175.26" y="-48.26" rot="R90"/>
 <instance part="R13" gate="G$1" x="175.26" y="-60.96" rot="R90"/>
+<instance part="SUPPLY14" gate="GND" x="157.48" y="-30.48"/>
 </instances>
 <busses>
@@
 <pinref part="U$1" gate="G$1" pin="PB4(ADC11)"/>
 <wire x1="134.62" y1="38.1" x2="165.1" y2="38.1" width="0.1524" layer="91"/>
-<wire x1="165.1" y1="38.1" x2="165.1" y2="-40.64" width="0.1524" layer="91"/>
+<wire x1="165.1" y1="38.1" x2="165.1" y2="0" width="0.1524" layer="91"/>
 <pinref part="R9" gate="G$1" pin="2"/>
-<wire x1="165.1" y1="-40.64" x2="175.26" y2="-40.64" width="0.1524" layer="91"/>
-<wire x1="175.26" y1="-40.64" x2="175.26" y2="-43.18" width="0.1524" layer="91"/>
+<wire x1="165.1" y1="0" x2="175.26" y2="-10.16" width="0.1524" layer="91"/>
+<wire x1="175.26" y1="-10.16" x2="175.26" y2="-43.18" width="0.1524" layer="91"/>
 </segment>
 </net>
@@
 <pinref part="SUPPLY11" gate="GND" pin="GND"/>
 <wire x1="175.26" y1="-66.04" x2="175.26" y2="-68.58" width="0.1524" layer="91"/>
+</segment>
+<segment>
+<pinref part="R10" gate="G$1" pin="1"/>
+<pinref part="SUPPLY14" gate="GND" pin="GND"/>
+<wire x1="157.48" y1="-25.4" x2="157.48" y2="-27.94" width="0.1524" layer="91"/>
 </segment>
 </net>
@@
 </segment>
 <segment>
-<pinref part="R11" gate="G$1" pin="2"/>
-<wire x1="198.12" y1="-12.7" x2="198.12" y2="-7.62" width="0.1524" layer="91"/>
-</segment>
-<segment>
 <pinref part="D1" gate="G$1" pin="C"/>
 <pinref part="+5V5" gate="1" pin="+5V"/>
@@
 </segment>
 <segment>
-<pinref part="R10" gate="G$1" pin="2"/>
-<wire x1="172.72" y1="-12.7" x2="172.72" y2="-7.62" width="0.1524" layer="91"/>
-<pinref part="Q1" gate="G$1" pin="G"/>
-<wire x1="185.42" y1="-15.24" x2="185.42" y2="-12.7" width="0.1524" layer="91"/>
-<wire x1="185.42" y1="-12.7" x2="172.72" y2="-12.7" width="0.1524" layer="91"/>
-<junction x="172.72" y="-12.7"/>
-</segment>
-<segment>
 <wire x1="185.42" y1="172.72" x2="185.42" y2="157.48" width="0.1524" layer="91"/>
 <wire x1="185.42" y1="157.48" x2="220.98" y2="157.48" width="0.1524" layer="91"/>
@@
 <pinref part="U$1" gate="G$1" pin="PD3(INT3/TXD1)"/>
 <wire x1="134.62" y1="12.7" x2="147.32" y2="12.7" width="0.1524" layer="91"/>
-<wire x1="147.32" y1="12.7" x2="160.02" y2="0" width="0.1524" layer="91"/>
-<wire x1="160.02" y1="0" x2="160.02" y2="-27.94" width="0.1524" layer="91"/>
-<wire x1="160.02" y1="-27.94" x2="198.12" y2="-27.94" width="0.1524" layer="91"/>
-<pinref part="Q1" gate="G$1" pin="D"/>
-<pinref part="R11" gate="G$1" pin="1"/>
-<wire x1="190.5" y1="-22.86" x2="198.12" y2="-22.86" width="0.1524" layer="91"/>
-<wire x1="198.12" y1="-27.94" x2="198.12" y2="-22.86" width="0.1524" layer="91"/>
-<junction x="198.12" y="-22.86"/>
+<wire x1="147.32" y1="12.7" x2="157.48" y2="2.54" width="0.1524" layer="91"/>
+<pinref part="R11" gate="G$1" pin="2"/>
+<wire x1="157.48" y1="-2.54" x2="157.48" y2="2.54" width="0.1524" layer="91"/>
 </segment>
 </net>
@@
 <wire x1="83.82" y1="-12.7" x2="88.9" y2="-7.62" width="0.1524" layer="91"/>
 <wire x1="88.9" y1="-7.62" x2="149.86" y2="-7.62" width="0.1524" layer="91"/>
-<wire x1="149.86" y1="-7.62" x2="154.94" y2="-12.7" width="0.1524" layer="91"/>
-<wire x1="154.94" y1="-12.7" x2="154.94" y2="-20.32" width="0.1524" layer="91"/>
-<wire x1="154.94" y1="-20.32" x2="157.48" y2="-22.86" width="0.1524" layer="91"/>
-<pinref part="R10" gate="G$1" pin="1"/>
-<wire x1="157.48" y1="-22.86" x2="172.72" y2="-22.86" width="0.1524" layer="91"/>
-<pinref part="Q1" gate="G$1" pin="S"/>
-<wire x1="172.72" y1="-22.86" x2="180.34" y2="-22.86" width="0.1524" layer="91"/>
-<junction x="172.72" y="-22.86"/>
-</segment>
-</net>
+<wire x1="149.86" y1="-7.62" x2="149.86" y2="-15.24" width="0.1524" layer="91"/>
+<pinref part="R10" gate="G$1" pin="2"/>
+<wire x1="149.86" y1="-15.24" x2="157.48" y2="-15.24" width="0.1524" layer="91"/>
+<pinref part="R11" gate="G$1" pin="1"/>
+<wire x1="157.48" y1="-15.24" x2="157.48" y2="-12.7" width="0.1524" layer="91"/>
+<junction x="157.48" y="-15.24"/>
+</segment>
+</net>

Commit message: Last sleep mode tweak, added line from BT LE to CAN1INT to wake the MCU up via BT
Parts:
- added Q1: MOSFET-NCHANNEL2N7002PW, SparkFun-DiscreteSemi:MOSFET-NCHANNEL2N7002PW
- L1: value 47uH -> 68uH
Connections:
- new net N$33: Q1.G, U1.P0_1
- net +5V: no longer L1.2
- net CAN1_INT: now also Q1.D
- net GND: now also Q1.S
Other:
- moved on the sheet: L1, R10, R11
Changed lines of the file:
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@@
 <part name="IC5" library="lm2674" deviceset="LM2674" device=""/>
 <part name="C11" library="resistor" deviceset="C-US" device="C0603" value=".01 uF"/>
-<part name="L1" library="inductor-bourns" deviceset="SDR0604" device="" value="47uH"/>
+<part name="L1" library="inductor-bourns" deviceset="SDR0604" device="" value="68uH"/>
 <part name="IC6" library="dp_devices" deviceset="IC_MEM_23LC1024" device=""/>
 <part name="C5" library="resistor" deviceset="C-US" device="C0603" value="0.1uF"/>
@@
 <part name="C13" library="resistor" deviceset="C-US" device="C0603" value="20pF"/>
 <part name="SUPPLY6" library="supply2" deviceset="GND" device=""/>
-<part name="D3" library="adafruit" deviceset="DIODE" device="SOD-323F"/>
 <part name="D2" library="adafruit" deviceset="DIODE" device="SOD-323F"/>
 <part name="SUPPLY11" library="supply2" deviceset="GND" device=""/>
@@
 <part name="R13" library="resistor" deviceset="R-US_" device="M0805" value="10k"/>
 <part name="SUPPLY14" library="supply2" deviceset="GND" device=""/>
+<part name="D3" library="adafruit" deviceset="DIODE" device="SOD-323F"/>
+<part name="Q1" library="SparkFun-DiscreteSemi" deviceset="MOSFET-NCHANNEL" device="2N7002PW"/>
+<part name="SUPPLY15" library="supply2" deviceset="GND" device=""/>
 </parts>
 <sheets>
@@
 <instance part="F1" gate="G$1" x="-20.32" y="83.82" rot="R180"/>
 <instance part="SUPPLY5" gate="GND" x="66.04" y="-43.18"/>
-<instance part="R10" gate="G$1" x="157.48" y="-20.32" rot="R90"/>
-<instance part="R11" gate="G$1" x="157.48" y="-7.62" rot="R90"/>
+<instance part="R10" gate="G$1" x="157.48" y="-17.78" rot="R90"/>
+<instance part="R11" gate="G$1" x="157.48" y="-5.08" rot="R90"/>
 <instance part="BT" gate="G$1" x="142.24" y="-58.42" rot="R90"/>
 <instance part="R12" gate="G$1" x="152.4" y="-63.5" rot="R90"/>
@@
 <instance part="IC5" gate="G$1" x="15.24" y="96.52" rot="R180"/>
 <instance part="C11" gate="G$1" x="33.02" y="91.44"/>
-<instance part="L1" gate="G$1" x="30.48" y="78.74"/>
+<instance part="L1" gate="G$1" x="25.4" y="78.74"/>
 <instance part="IC6" gate="IC" x="210.82" y="139.7" rot="R90"/>
 <instance part="IC6" gate="SUP" x="73.66" y="134.62"/>
@@
 <instance part="C13" gate="G$1" x="68.58" y="33.02" rot="R270"/>
 <instance part="SUPPLY6" gate="GND" x="53.34" y="26.67"/>
-<instance part="D3" gate="G$1" x="-20.32" y="93.98" rot="R270"/>
 <instance part="D2" gate="G$1" x="15.24" y="73.66" rot="R90"/>
 <instance part="SUPPLY11" gate="GND" x="175.26" y="-71.12"/>
 <instance part="R9" gate="G$1" x="175.26" y="-48.26" rot="R90"/>
 <instance part="R13" gate="G$1" x="175.26" y="-60.96" rot="R90"/>
-<instance part="SUPPLY14" gate="GND" x="157.48" y="-30.48"/>
+<instance part="SUPPLY14" gate="GND" x="157.48" y="-27.94"/>
+<instance part="D3" gate="G$1" x="-20.32" y="93.98" rot="R270"/>
+<instance part="Q1" gate="G$1" x="203.2" y="-40.64" rot="R270"/>
+<instance part="SUPPLY15" gate="GND" x="195.58" y="-45.72"/>
 </instances>
 <busses>
@@
 <pinref part="CAN-CNT-1" gate="D" pin="INT"/>
 <wire x1="213.36" y1="96.52" x2="238.76" y2="96.52" width="0.1524" layer="91"/>
+<pinref part="Q1" gate="G$1" pin="D"/>
+<wire x1="208.28" y1="-40.64" x2="213.36" y2="-40.64" width="0.1524" layer="91"/>
+<wire x1="213.36" y1="-40.64" x2="213.36" y2="5.08" width="0.1524" layer="91"/>
+<junction x="213.36" y="5.08"/>
 </segment>
 </net>
@@
 <pinref part="SUPPLY11" gate="GND" pin="GND"/>
 <wire x1="175.26" y1="-66.04" x2="175.26" y2="-68.58" width="0.1524" layer="91"/>
+<wire x1="175.26" y1="-66.04" x2="213.36" y2="-66.04" width="0.1524" layer="91"/>
+<junction x="175.26" y="-66.04"/>
 </segment>
 <segment>
 <pinref part="R10" gate="G$1" pin="1"/>
 <pinref part="SUPPLY14" gate="GND" pin="GND"/>
-<wire x1="157.48" y1="-25.4" x2="157.48" y2="-27.94" width="0.1524" layer="91"/>
+<wire x1="157.48" y1="-22.86" x2="157.48" y2="-25.4" width="0.1524" layer="91"/>
+</segment>
+<segment>
+<pinref part="Q1" gate="G$1" pin="S"/>
+<wire x1="198.12" y1="-40.64" x2="195.58" y2="-40.64" width="0.1524" layer="91"/>
+<wire x1="195.58" y1="-40.64" x2="195.58" y2="-43.18" width="0.1524" layer="91"/>
+<pinref part="SUPPLY15" gate="GND" pin="GND"/>
 </segment>
 </net>
@@
 <wire x1="27.94" y1="101.6" x2="45.72" y2="101.6" width="0.1524" layer="91"/>
 <wire x1="45.72" y1="101.6" x2="45.72" y2="78.74" width="0.1524" layer="91"/>
-<pinref part="L1" gate="G$1" pin="2"/>
-<wire x1="45.72" y1="78.74" x2="35.56" y2="78.74" width="0.1524" layer="91"/>
 </segment>
 <segment>
@@
 <wire x1="147.32" y1="12.7" x2="157.48" y2="2.54" width="0.1524" layer="91"/>
 <pinref part="R11" gate="G$1" pin="2"/>
-<wire x1="157.48" y1="-2.54" x2="157.48" y2="2.54" width="0.1524" layer="91"/>
+<wire x1="157.48" y1="0" x2="157.48" y2="2.54" width="0.1524" layer="91"/>
 </segment>
 </net>
@@
 <wire x1="83.82" y1="-12.7" x2="88.9" y2="-7.62" width="0.1524" layer="91"/>
 <wire x1="88.9" y1="-7.62" x2="149.86" y2="-7.62" width="0.1524" layer="91"/>
-<wire x1="149.86" y1="-7.62" x2="149.86" y2="-15.24" width="0.1524" layer="91"/>
+<wire x1="149.86" y1="-7.62" x2="149.86" y2="-12.7" width="0.1524" layer="91"/>
 <pinref part="R10" gate="G$1" pin="2"/>
-<wire x1="149.86" y1="-15.24" x2="157.48" y2="-15.24" width="0.1524" layer="91"/>
+<wire x1="149.86" y1="-12.7" x2="157.48" y2="-12.7" width="0.1524" layer="91"/>
 <pinref part="R11" gate="G$1" pin="1"/>
-<wire x1="157.48" y1="-15.24" x2="157.48" y2="-12.7" width="0.1524" layer="91"/>
-<junction x="157.48" y="-15.24"/>
+<wire x1="157.48" y1="-12.7" x2="157.48" y2="-10.16" width="0.1524" layer="91"/>
+<junction x="157.48" y="-12.7"/>
 </segment>
 </net>
@@
 <wire x1="2.54" y1="78.74" x2="15.24" y2="78.74" width="0.1524" layer="91"/>
 <pinref part="C11" gate="G$1" pin="2"/>
-<wire x1="15.24" y1="78.74" x2="25.4" y2="78.74" width="0.1524" layer="91"/>
+<wire x1="15.24" y1="78.74" x2="20.32" y2="78.74" width="0.1524" layer="91"/>
 <wire x1="33.02" y1="86.36" x2="2.54" y2="86.36" width="0.1524" layer="91"/>
 <pinref part="L1" gate="G$1" pin="1"/>
@@
 </segment>
 </net>
-<net name="N$22" class="0">
-<segment>
-<pinref part="F1" gate="G$1" pin="2"/>
-<wire x1="-20.32" y1="88.9" x2="-20.32" y2="91.44" width="0.1524" layer="91"/>
-<pinref part="D3" gate="G$1" pin="C"/>
-</segment>
-</net>
 <net name="N$29" class="0">
 <segment>
@@
 </segment>
 </net>
+<net name="N$33" class="0">
+<segment>
+<pinref part="U1" gate="G$1" pin="P0_1"/>
+<wire x1="132.08" y1="-33.02" x2="203.2" y2="-33.02" width="0.1524" layer="91"/>
+<pinref part="Q1" gate="G$1" pin="G"/>
+</segment>
+</net>
+<net name="N$22" class="0">
+<segment>
+<pinref part="F1" gate="G$1" pin="2"/>
+<wire x1="-20.32" y1="88.9" x2="-20.32" y2="91.44" width="0.1524" layer="91"/>
+<pinref part="D3" gate="G$1" pin="C"/>
+</segment>
+</net>

Commit message: Fix missing trace on inductor
Connections:
- net +5V: now also L1.2
Changed lines of the file:
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@@
 <wire x1="27.94" y1="101.6" x2="45.72" y2="101.6" width="0.1524" layer="91"/>
 <wire x1="45.72" y1="101.6" x2="45.72" y2="78.74" width="0.1524" layer="91"/>
+<pinref part="L1" gate="G$1" pin="2"/>
+<wire x1="30.48" y1="78.74" x2="45.72" y2="78.74" width="0.1524" layer="91"/>
 </segment>
 <segment>

Commit message: switched to LM3480IM3-5.0
Parts:
- removed C11: .01 uF, resistor:C-USC0603
- removed D3: (no value), adafruit:DIODESOD-323F
- removed IC5: (no value), lm2674:LM2674
- removed L1: 68uH, inductor-bourns:SDR0604
- added IC1: LM3480, CustomParts_CBT:LM3480
- C1: value 22uF -> 0.1uF; device resistor:C-USC0805 -> resistor:C-USC0603
- C2: value 47uF -> 0.1uF; device resistor:C-USC1206 -> resistor:C-USC0603
- renumbered U$11 to Q2, U$2 to Q0
Connections:
- removed net N$22: D3.C, F1.2
- removed net N$34: C11.1, IC5.CB
- net +12V: now also F1.2; no longer D3.A
- net +5V: now also IC1.VO; no longer IC5.FB, L1.2
- net GND: now also IC1.GND; no longer D2.A, IC5.GND
- net N$15: now also D2.A, F1.1; no longer C11.2, D2.C, IC5.VSW, L1.1
- net SUPPLY: now also D2.C, IC1.VI; no longer F1.1, IC5.VIN
Other:
- moved on the sheet: C1, C2, D2, F1

Commit message: switched to TPS70950 LDO Linear Regulator
Parts:
- removed D2: (no value), adafruit:DIODESOD-323F
- removed F1: POLYFUSE, rcl:L-EUL1812
- C1: value 0.1uF -> 1uF
- C2: value 0.1uF -> 2.2uF
- IC1: value LM3480 -> TPS709-50; device CustomParts_CBT:LM3480 -> CustomParts_CBT:TPS709-50
Connections:
- removed net N$15: D2.A, F1.1
- removed net SUPPLY: C1.1, D2.C, IC1.VI
- net +12V: now also C1.1, IC1.VI; no longer F1.2

Commit message: Some part name changes
Parts:
- renumbered CAN-CNT-1 to CC1, CAN-CNT-2 to CC2, CAN-CNT-3 to CC3, CAN-TRNS-1 to CT1, CAN-TRNS-2 to CT2, CAN-TRNS-3 to CT3, CAN1-TRM to R14, CAN2-TRM to R15, CAN3-TRM to R16
